File: docs/projects/esrmeter/esrmeter.brd (EAGLE design)
At the start: 58.1 x 52.1 mm, 18 parts, among them IC2 TL072P

Commit message: esrmeter: modify schematic
Connections:
- removed net N$4: IC2.3, IC2.7, R1.2
- net A4: now also IC2.3, IC2.7, R1.2
Routing:
- net A4: track 0.00 -> 36.6 mm, vias 0 -> 4
- net N$4: track 13.8 -> 0.00 mm, vias 2 -> 0
- net GND: track 142.2 -> 143.3 mm
Other:
- board text added: "A4"
Changed lines of the file:
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@@
 <text x="33.02" y="45.72" size="2.54" layer="110">Capacitor</text>
 <text x="35.56" y="5.08" size="1.778" layer="110">D9</text>
-<text x="71.12" y="5.08" size="1.778" layer="110">A5</text>
+<text x="74.93" y="5.08" size="1.778" layer="110">A5</text>
 <hole x="58.42" y="20.32" drill="1.5"/>
 <hole x="76.2" y="22.86" drill="1.5"/>
@@
 <hole x="81.28" y="25.4" drill="1.5"/>
 <hole x="81.28" y="7.62" drill="1.5"/>
-<hole x="78.74" y="17.78" drill="1.5"/>
 <hole x="50.8" y="40.64" drill="1.5"/>
 <hole x="53.34" y="40.64" drill="1.5"/>
@@
 <hole x="48.26" y="40.64" drill="1.5"/>
 <hole x="66.04" y="40.64" drill="1.5"/>
+<text x="72.39" y="11.43" size="1.778" layer="110">A4</text>
 </plain>
 <attributes>
@@
 <wire x1="55.88" y1="22.86" x2="55.88" y2="25.4" width="0.4064" layer="16"/>
 <wire x1="55.88" y1="25.4" x2="55.88" y2="38.1" width="0.4064" layer="16"/>
-<wire x1="55.88" y1="7.62" x2="86.36" y2="7.62" width="0.4064" layer="1"/>
+<wire x1="55.88" y1="7.62" x2="57.15" y2="8.89" width="0.4064" layer="1"/>
+<wire x1="57.15" y1="8.89" x2="85.09" y2="8.89" width="0.4064" layer="1"/>
+<wire x1="85.09" y1="8.89" x2="86.36" y2="7.62" width="0.4064" layer="1"/>
 <wire x1="55.88" y1="38.1" x2="55.88" y2="43.18" width="0.4064" layer="16"/>
 <wire x1="55.88" y1="43.18" x2="55.88" y2="45.72" width="0.4064" layer="16"/>
@@
 <signal name="A4">
 <contactref element="PC" pad="6"/>
+<contactref element="IC2" pad="7"/>
+<contactref element="R1" pad="2"/>
+<contactref element="IC2" pad="3"/>
+<wire x1="76.2" y1="27.94" x2="76.2" y2="33.02" width="0.4064" layer="16"/>
+<wire x1="78.74" y1="20.32" x2="78.74" y2="22.86" width="0.4064" layer="16"/>
+<wire x1="76.2" y1="25.4" x2="76.2" y2="27.94" width="0.4064" layer="16"/>
+<wire x1="78.74" y1="22.86" x2="76.2" y2="25.4" width="0.4064" layer="1"/>
+<via x="78.74" y="22.86" extent="1-16" drill="0.6" shape="square"/>
+<via x="76.2" y="25.4" extent="1-16" drill="0.6" shape="square"/>
+<wire x1="73.66" y1="2.54" x2="73.66" y2="7.62" width="0.4064" layer="16"/>
+<wire x1="78.74" y1="20.32" x2="78.74" y2="7.62" width="0.4064" layer="16"/>
+<via x="73.66" y="7.62" extent="1-16" drill="0.6" shape="square"/>
+<via x="78.74" y="7.62" extent="1-16" drill="0.6" shape="square"/>
+<wire x1="73.66" y1="7.62" x2="78.74" y2="7.62" width="0.4064" layer="1"/>
 </signal>
 <signal name="A5">
@@
 <wire x1="78.74" y1="33.02" x2="78.74" y2="38.1" width="0.4064" layer="16"/>
 </signal>
-<signal name="N$4">
-<contactref element="IC2" pad="7"/>
-<contactref element="R1" pad="2"/>
-<contactref element="IC2" pad="3"/>
-<wire x1="76.2" y1="27.94" x2="76.2" y2="33.02" width="0.4064" layer="16"/>
-<wire x1="78.74" y1="20.32" x2="78.74" y2="22.86" width="0.4064" layer="16"/>
-<wire x1="76.2" y1="25.4" x2="76.2" y2="27.94" width="0.4064" layer="16"/>
-<wire x1="78.74" y1="22.86" x2="76.2" y2="25.4" width="0.4064" layer="1"/>
-<via x="78.74" y="22.86" extent="1-16" drill="0.6" shape="square"/>
-<via x="76.2" y="25.4" extent="1-16" drill="0.6" shape="square"/>
-</signal>
 <signal name="N$5">
