File: docs/projects/buzzer/buzzer.brd (EAGLE design)
At the start: 48.2 x 27.6 mm, 12 parts, among them T1 BC238

Commit message: fix airwires
Changed lines of the file:
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@@
 <contactref element="R2" pad="2"/>
 <contactref element="R3" pad="E"/>
-<wire x1="20.32" y1="22.86" x2="48.26" y2="22.86" width="0.4064" layer="16"/>
+<wire x1="27.94" y1="22.86" x2="48.26" y2="22.86" width="0.4064" layer="16"/>
 <wire x1="20.32" y1="25.4" x2="20.32" y2="27.94" width="0.4064" layer="1"/>
 <wire x1="20.32" y1="22.86" x2="20.32" y2="25.4" width="0.4064" layer="1"/>
@@
 <wire x1="20.32" y1="12.7" x2="20.32" y2="15.24" width="0.4064" layer="1"/>
 <wire x1="20.32" y1="10.16" x2="20.32" y2="12.7" width="0.4064" layer="1"/>
-<wire x1="20.32" y1="22.86" x2="27.94" y2="22.86" width="0" layer="19" extent="16-16"/>
+<wire x1="20.32" y1="22.86" x2="27.94" y2="22.86" width="0.4064" layer="16"/>
 </signal>
 <signal name="N$2">
