File: docs/projects/extpower/extpower.brd (EAGLE design)
At the start: 48.2 x 27.6 mm, 11 parts, among them IC1 7805T

Commit message: fix airwires
Routing:
- net GND: track 83.8 -> 99.1 mm
- net +5V: track 17.8 -> 33.0 mm
- net N$4: track 0.00 -> 2.54 mm
Changed lines of the file:
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@@
 <contactref element="LED4" pad="A"/>
 <contactref element="R8" pad="2"/>
-<wire x1="58.42" y1="7.62" x2="55.88" y2="7.62" width="0" layer="19" extent="1-1"/>
+<wire x1="55.88" y1="7.62" x2="58.42" y2="7.62" width="0.4064" layer="16"/>
 </signal>
 <signal name="GND">
@@
 <wire x1="22.86" y1="10.16" x2="20.32" y2="10.16" width="0.4064" layer="16"/>
 <wire x1="20.32" y1="10.16" x2="20.32" y2="20.32" width="0.4064" layer="1"/>
-<wire x1="43.18" y1="10.16" x2="58.42" y2="10.16" width="0" layer="19" extent="16-16"/>
 <via x="43.18" y="10.16" extent="1-16" drill="0.6" shape="square"/>
 <via x="43.18" y="5.08" extent="1-16" drill="0.6" shape="square"/>
 <via x="20.32" y="10.16" extent="1-16" drill="0.6" shape="square"/>
 <via x="20.32" y="20.32" extent="1-16" drill="0.6" shape="square"/>
+<wire x1="58.42" y1="10.16" x2="43.18" y2="10.16" width="0.4064" layer="16"/>
 </signal>
 <signal name="+5V">
@@
 <wire x1="22.86" y1="7.62" x2="27.94" y2="7.62" width="0.4064" layer="16"/>
 <wire x1="27.94" y1="7.62" x2="30.48" y2="7.62" width="0.4064" layer="16"/>
-<wire x1="30.48" y1="7.62" x2="45.72" y2="7.62" width="0" layer="19" extent="1-1"/>
+<wire x1="45.72" y1="7.62" x2="30.48" y2="7.62" width="0.4064" layer="16"/>
 </signal>
 <signal name="N$2">
@@
 <wire x1="27.94" y1="27.94" x2="55.88" y2="27.94" width="0.4064" layer="16"/>
 <wire x1="27.94" y1="25.4" x2="27.94" y2="27.94" width="0.4064" layer="1"/>
-<wire x1="55.88" y1="20.32" x2="53.34" y2="20.32" width="0.4064" layer="16"/>
 <wire x1="55.88" y1="27.94" x2="55.88" y2="20.32" width="0.4064" layer="1"/>
-<wire x1="53.34" y1="20.32" x2="53.8" y2="20.32" width="0" layer="19" extent="16-16"/>
 <via x="27.94" y="25.4" extent="1-16" drill="0.6" shape="square"/>
 <via x="27.94" y="27.94" extent="1-16" drill="0.6" shape="square"/>
 <via x="55.88" y="27.94" extent="1-16" drill="0.6" shape="square"/>
 <via x="55.88" y="20.32" extent="1-16" drill="0.6" shape="square"/>
+<wire x1="53.8" y1="20.32" x2="55.88" y2="20.32" width="0.4064" layer="16"/>
+<wire x1="53.8" y1="20.32" x2="53.34" y2="20.32" width="0.4064" layer="16"/>
 </signal>
 </signals>
