File: docs/projects/r2r_ladder_dac/r2r_ladder_dac.brd (EAGLE design)
At the start: 48.2 x 27.6 mm, 25 parts, among them IC1 LM358N

Commit message: fix airwires
Routing:
- net GND: track 0.00 -> 61.6 mm
- net +5V: track 0.00 -> 31.5 mm
- net N$17: track 0.00 -> 15.8 mm, vias 0 -> 1
- net N$8: track 0.00 -> 10.7 mm
- net N$4: track 0.00 -> 8.89 mm
- net N$19: track 0.00 -> 7.62 mm
- net N$9: track 0.00 -> 7.62 mm
- net N$16: track 0.00 -> 7.62 mm
- net N$15: track 0.00 -> 7.62 mm
- net N$14: track 0.00 -> 7.62 mm
- net N$13: track 0.00 -> 7.62 mm
- net N$12: track 0.00 -> 7.62 mm
- net N$11: track 0.00 -> 7.62 mm
- net N$10: track 0.00 -> 7.62 mm
- net N$18: track 0.00 -> 5.08 mm
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Changed lines of the file:
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@@
 <contactref element="R20" pad="1"/>
 <contactref element="IC1" pad="4"/>
-<wire x1="50.8" y1="15.24" x2="55.88" y2="16.51" width="0" layer="19" extent="1-1"/>
-<wire x1="53.34" y1="5.08" x2="50.8" y2="15.24" width="0" layer="19" extent="1-1"/>
-<wire x1="38.1" y1="3.81" x2="53.34" y2="5.08" width="0" layer="19" extent="1-1"/>
-<wire x1="12.7" y1="5.08" x2="38.1" y2="3.81" width="0" layer="19" extent="1-1"/>
+<wire x1="52.07" y1="16.51" x2="50.8" y2="15.24" width="0.254" layer="16"/>
+<wire x1="55.88" y1="16.51" x2="52.07" y2="16.51" width="0.254" layer="16"/>
+<wire x1="30.48" y1="5.08" x2="35.56" y2="5.08" width="0.254" layer="16"/>
+<wire x1="35.56" y1="5.08" x2="53.34" y2="5.08" width="0.254" layer="16"/>
+<wire x1="29.21" y1="6.35" x2="30.48" y2="5.08" width="0.254" layer="16"/>
+<wire x1="21.59" y1="6.35" x2="29.21" y2="6.35" width="0.254" layer="16"/>
+<wire x1="20.32" y1="5.08" x2="21.59" y2="6.35" width="0.254" layer="16"/>
+<wire x1="12.7" y1="5.08" x2="20.32" y2="5.08" width="0.254" layer="16"/>
+<wire x1="36.83" y1="3.81" x2="38.1" y2="3.81" width="0.254" layer="16"/>
+<wire x1="35.56" y1="5.08" x2="36.83" y2="3.81" width="0.254" layer="16"/>
+<wire x1="52.07" y1="13.97" x2="50.8" y2="15.24" width="0.254" layer="1"/>
+<wire x1="52.07" y1="12.7" x2="52.07" y2="13.97" width="0.254" layer="1"/>
+<wire x1="53.34" y1="11.43" x2="52.07" y2="12.7" width="0.254" layer="1"/>
+<wire x1="53.34" y1="5.08" x2="53.34" y2="11.43" width="0.254" layer="1"/>
 </signal>
 <signal name="+5V">
 <contactref element="SV1" pad="2"/>
 <contactref element="IC1" pad="8"/>
-<wire x1="12.7" y1="7.62" x2="43.18" y2="7.62" width="0" layer="19" extent="1-1"/>
+<wire x1="30.48" y1="7.62" x2="43.18" y2="7.62" width="0.254" layer="16"/>
+<wire x1="29.21" y1="8.89" x2="30.48" y2="7.62" width="0.254" layer="16"/>
+<wire x1="21.59" y1="8.89" x2="29.21" y2="8.89" width="0.254" layer="16"/>
+<wire x1="20.32" y1="7.62" x2="21.59" y2="8.89" width="0.254" layer="16"/>
+<wire x1="12.7" y1="7.62" x2="20.32" y2="7.62" width="0.254" layer="16"/>
 </signal>
 <signal name="N$1">
@@
 <contactref element="R2" pad="1"/>
 <contactref element="R11" pad="2"/>
-<wire x1="33.02" y1="22.86" x2="35.56" y2="22.86" width="0" layer="19" extent="1-1"/>
-<wire x1="30.48" y1="22.86" x2="33.02" y2="22.86" width="0" layer="19" extent="1-1"/>
+<wire x1="30.48" y1="22.86" x2="33.02" y2="22.86" width="0.254" layer="1"/>
+<wire x1="33.02" y1="22.86" x2="35.56" y2="22.86" width="0.254" layer="1"/>
 </signal>
 <signal name="N$2">
@@
 <contactref element="R3" pad="1"/>
 <contactref element="R8" pad="2"/>
-<wire x1="33.02" y1="20.32" x2="35.56" y2="20.32" width="0" layer="19" extent="1-1"/>
-<wire x1="30.48" y1="20.32" x2="33.02" y2="20.32" width="0" layer="19" extent="1-1"/>
+<wire x1="30.48" y1="20.32" x2="33.02" y2="20.32" width="0.254" layer="1"/>
+<wire x1="33.02" y1="20.32" x2="35.56" y2="20.32" width="0.254" layer="1"/>
 </signal>
 <signal name="N$3">
@@
 <contactref element="R4" pad="1"/>
 <contactref element="R12" pad="2"/>
-<wire x1="33.02" y1="17.78" x2="35.56" y2="17.78" width="0" layer="19" extent="1-1"/>
-<wire x1="30.48" y1="17.78" x2="33.02" y2="17.78" width="0" layer="19" extent="1-1"/>
+<wire x1="30.48" y1="17.78" x2="33.02" y2="17.78" width="0.254" layer="1"/>
+<wire x1="33.02" y1="17.78" x2="35.56" y2="17.78" width="0.254" layer="1"/>
 </signal>
 <signal name="N$5">
@@
 <contactref element="R5" pad="1"/>
 <contactref element="R13" pad="2"/>
-<wire x1="33.02" y1="15.24" x2="35.56" y2="15.24" width="0" layer="19" extent="1-1"/>
-<wire x1="30.48" y1="15.24" x2="33.02" y2="15.24" width="0" layer="19" extent="1-1"/>
+<wire x1="30.48" y1="15.24" x2="33.02" y2="15.24" width="0.254" layer="1"/>
+<wire x1="33.02" y1="15.24" x2="35.56" y2="15.24" width="0.254" layer="1"/>
 </signal>
 <signal name="N$6">
@@
 <contactref element="R6" pad="1"/>
 <contactref element="R14" pad="2"/>
-<wire x1="33.02" y1="12.7" x2="35.56" y2="12.7" width="0" layer="19" extent="1-1"/>
-<wire x1="30.48" y1="12.7" x2="33.02" y2="12.7" width="0" layer="19" extent="1-1"/>
+<wire x1="30.48" y1="12.7" x2="33.02" y2="12.7" width="0.254" layer="1"/>
+<wire x1="33.02" y1="12.7" x2="35.56" y2="12.7" width="0.254" layer="1"/>
 </signal>
 <signal name="N$7">
@@
 <contactref element="R7" pad="2"/>
 <contactref element="R10" pad="2"/>
-<wire x1="33.02" y1="25.4" x2="35.56" y2="25.4" width="0" layer="19" extent="1-1"/>
-<wire x1="30.48" y1="25.4" x2="33.02" y2="25.4" width="0" layer="19" extent="1-1"/>
+<wire x1="30.48" y1="25.4" x2="33.02" y2="25.4" width="0.254" layer="1"/>
+<wire x1="33.02" y1="25.4" x2="35.56" y2="25.4" width="0.254" layer="1"/>
 </signal>
 <signal name="N$4">
@@
 <contactref element="R9" pad="1"/>
 <contactref element="R15" pad="2"/>
-<wire x1="38.1" y1="26.67" x2="35.56" y2="27.94" width="0" layer="19" extent="1-1"/>
-<wire x1="30.48" y1="27.94" x2="35.56" y2="27.94" width="0" layer="19" extent="1-1"/>
+<wire x1="30.48" y1="27.94" x2="35.56" y2="27.94" width="0.254" layer="16"/>
+<wire x1="38.1" y1="27.94" x2="38.1" y2="26.67" width="0.254" layer="16"/>
+<wire x1="35.56" y1="27.94" x2="38.1" y2="27.94" width="0.254" layer="16"/>
 </signal>
 <signal name="N$8">
@@
 <contactref element="R16" pad="2"/>
 <contactref element="R17" pad="1"/>
-<wire x1="35.56" y1="10.16" x2="40.64" y2="8.89" width="0" layer="19" extent="1-1"/>
-<wire x1="30.48" y1="10.16" x2="35.56" y2="10.16" width="0" layer="19" extent="1-1"/>
+<wire x1="30.48" y1="10.16" x2="35.56" y2="10.16" width="0.254" layer="16"/>
+<wire x1="36.83" y1="8.89" x2="40.64" y2="8.89" width="0.254" layer="16"/>
+<wire x1="35.56" y1="10.16" x2="36.83" y2="8.89" width="0.254" layer="16"/>
 </signal>
 <signal name="N$9">
 <contactref element="R15" pad="1"/>
 <contactref element="SV1" pad="10"/>
-<wire x1="12.7" y1="27.94" x2="20.32" y2="27.94" width="0" layer="19" extent="1-1"/>
+<wire x1="12.7" y1="27.94" x2="20.32" y2="27.94" width="0.254" layer="16"/>
 </signal>
 <signal name="N$10">
 <contactref element="SV1" pad="9"/>
 <contactref element="R10" pad="1"/>
-<wire x1="12.7" y1="25.4" x2="20.32" y2="25.4" width="0" layer="19" extent="1-1"/>
+<wire x1="12.7" y1="25.4" x2="20.32" y2="25.4" width="0.254" layer="16"/>
 </signal>
 <signal name="N$11">
 <contactref element="SV1" pad="8"/>
 <contactref element="R11" pad="1"/>
-<wire x1="12.7" y1="22.86" x2="20.32" y2="22.86" width="0" layer="19" extent="1-1"/>
+<wire x1="12.7" y1="22.86" x2="20.32" y2="22.86" width="0.254" layer="16"/>
 </signal>
 <signal name="N$12">
 <contactref element="SV1" pad="7"/>
 <contactref element="R8" pad="1"/>
-<wire x1="12.7" y1="20.32" x2="20.32" y2="20.32" width="0" layer="19" extent="1-1"/>
+<wire x1="12.7" y1="20.32" x2="20.32" y2="20.32" width="0.254" layer="16"/>
 </signal>
 <signal name="N$13">
 <contactref element="SV1" pad="6"/>
 <contactref element="R12" pad="1"/>
-<wire x1="12.7" y1="17.78" x2="20.32" y2="17.78" width="0" layer="19" extent="1-1"/>
+<wire x1="12.7" y1="17.78" x2="20.32" y2="17.78" width="0.254" layer="16"/>
 </signal>
 <signal name="N$14">
 <contactref element="SV1" pad="5"/>
 <contactref element="R13" pad="1"/>
-<wire x1="12.7" y1="15.24" x2="20.32" y2="15.24" width="0" layer="19" extent="1-1"/>
+<wire x1="12.7" y1="15.24" x2="20.32" y2="15.24" width="0.254" layer="16"/>
 </signal>
 <signal name="N$15">
 <contactref element="SV1" pad="4"/>
 <contactref element="R14" pad="1"/>
-<wire x1="12.7" y1="12.7" x2="20.32" y2="12.7" width="0" layer="19" extent="1-1"/>
+<wire x1="12.7" y1="12.7" x2="20.32" y2="12.7" width="0.254" layer="16"/>
 </signal>
 <signal name="N$16">
 <contactref element="SV1" pad="3"/>
 <contactref element="R16" pad="1"/>
-<wire x1="12.7" y1="10.16" x2="20.32" y2="10.16" width="0" layer="19" extent="1-1"/>
+<wire x1="12.7" y1="10.16" x2="20.32" y2="10.16" width="0.254" layer="16"/>
 </signal>
 <signal name="N$17">
@@
 <contactref element="R18" pad="1"/>
 <contactref element="IC1" pad="3"/>
-<wire x1="53.34" y1="15.24" x2="50.8" y2="12.7" width="0" layer="19" extent="1-1"/>
-<wire x1="40.64" y1="13.97" x2="53.34" y2="15.24" width="0" layer="19" extent="1-1"/>
+<wire x1="45.72" y1="13.97" x2="40.64" y2="13.97" width="0.254" layer="16"/>
+<wire x1="46.99" y1="12.7" x2="45.72" y2="13.97" width="0.254" layer="16"/>
+<wire x1="50.8" y1="12.7" x2="46.99" y2="12.7" width="0.254" layer="16"/>
+<wire x1="53.34" y1="12.7" x2="53.34" y2="15.24" width="0.254" layer="1"/>
+<wire x1="50.8" y1="12.7" x2="53.34" y2="12.7" width="0.254" layer="16"/>
+<via x="53.34" y="12.7" extent="1-16" drill="0.6096"/>
 </signal>
 <signal name="N$18">
 <contactref element="R19" pad="2"/>
 <contactref element="IC1" pad="1"/>
-<wire x1="50.8" y1="7.62" x2="55.88" y2="7.62" width="0" layer="19" extent="1-1"/>
+<wire x1="50.8" y1="7.62" x2="55.88" y2="7.62" width="0.254" layer="16"/>
 </signal>
 <signal name="N$19">
@@
 <contactref element="R19" pad="1"/>
 <contactref element="JP1" pad="2"/>
-<wire x1="55.88" y1="10.16" x2="58.42" y2="10.16" width="0" layer="19" extent="1-1"/>
-<wire x1="50.8" y1="10.16" x2="55.88" y2="10.16" width="0" layer="19" extent="1-1"/>
+<wire x1="50.8" y1="10.16" x2="55.88" y2="10.16" width="0.254" layer="16"/>
+<wire x1="55.88" y1="10.16" x2="58.42" y2="10.16" width="0.254" layer="1"/>
 </signal>
 <signal name="N$20">
 <contactref element="JP1" pad="1"/>
 <contactref element="R20" pad="2"/>
-<wire x1="55.88" y1="13.97" x2="58.42" y2="12.7" width="0" layer="19" extent="1-1"/>
+<wire x1="57.15" y1="12.7" x2="55.88" y2="13.97" width="0.254" layer="16"/>
+<wire x1="58.42" y1="12.7" x2="57.15" y2="12.7" width="0.254" layer="16"/>
 </signal>
 </signals>
