File: docs/projects/rs232/rs232.brd (EAGLE design)
At the start: 48.2 x 27.6 mm, 8 parts

Commit message: fix airwires
Routing:
- net GND: track 45.7 -> 63.5 mm, vias 0 -> 2
- net N$8: track 17.8 -> 0.00 mm, vias 2 -> 0
- net N$13: track 10.2 -> 0.00 mm, vias 2 -> 0
- net VCC: track 45.7 -> 55.9 mm, vias 0 -> 2
Changed lines of the file:
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@@
 <wire x1="17.78" y1="7.62" x2="27.94" y2="7.62" width="0.4064" layer="16"/>
 <wire x1="55.88" y1="25.4" x2="63.5" y2="25.4" width="0.4064" layer="16"/>
+<wire x1="55.88" y1="7.62" x2="55.88" y2="25.4" width="0.4064" layer="1"/>
+<via x="55.88" y="7.62" extent="1-16" drill="0.6" shape="square"/>
+<via x="55.88" y="25.4" extent="1-16" drill="0.6" shape="square"/>
 <wire x1="27.94" y1="7.62" x2="55.88" y2="7.62" width="0.4064" layer="16"/>
-<wire x1="55.88" y1="7.62" x2="55.88" y2="25.4" width="0" layer="19" extent="1-16"/>
 </signal>
 <signal name="VCC">
@@
 <wire x1="17.78" y1="10.16" x2="27.94" y2="10.16" width="0.4064" layer="16"/>
 <wire x1="53.34" y1="20.32" x2="63.5" y2="20.32" width="0.4064" layer="16"/>
-<wire x1="27.94" y1="10.16" x2="53.34" y2="10.16" width="0.4064" layer="16"/>
-<wire x1="53.34" y1="10.16" x2="53.34" y2="20.32" width="0" layer="19" extent="1-16"/>
+<wire x1="53.34" y1="10.16" x2="53.34" y2="20.32" width="0.4064" layer="1"/>
+<via x="53.34" y="10.16" extent="1-16" drill="0.6" shape="square"/>
+<via x="53.34" y="20.32" extent="1-16" drill="0.6" shape="square"/>
+<wire x1="53.34" y1="10.16" x2="27.94" y2="10.16" width="0.4064" layer="16"/>
 </signal>
 <signal name="RXD">
@@
 <wire x1="22.86" y1="27.94" x2="27.94" y2="27.94" width="0.4064" layer="16"/>
 </signal>
-<signal name="N$8">
-<wire x1="55.88" y1="7.62" x2="55.88" y2="25.4" width="0.4064" layer="1"/>
-<via x="55.88" y="7.62" extent="1-16" drill="0.6" shape="square"/>
-<via x="55.88" y="25.4" extent="1-16" drill="0.6" shape="square"/>
-</signal>
-<signal name="N$13">
-<wire x1="53.34" y1="10.16" x2="53.34" y2="20.32" width="0.4064" layer="1"/>
-<via x="53.34" y="10.16" extent="1-16" drill="0.6" shape="square"/>
-<via x="53.34" y="20.32" extent="1-16" drill="0.6" shape="square"/>
-</signal>
 </signals>
